Commit message: Adapted to the new version of Gazebo

File: src/ugv_roarm_moveit/config/roarm_m2/roarm_m2.ros2_control.xacro (robot description, xacro)
@@ -1,14 +1,19 @@
 <?xml version="1.0"?>
 <robot xmlns:xacro="http://www.ros.org/wiki/xacro">
-    <xacro:macro name="roarm_ros2_control" params="name initial_positions_file">
+    <xacro:macro name="roarm_ros2_control" params="use_gazebo GZ_VERSION initial_positions_file">
         <xacro:property name="initial_positions" value="${load_yaml(initial_positions_file)['initial_positions']}"/>
-        <ros2_control name="${name}" type="system">
+        <ros2_control name="RoarmHardware" type="system">
             <hardware>
-                <xacro:if value="${name== 'FakeSystem'}">
-                <plugin>mock_components/GenericSystem</plugin>
+              <xacro:unless value="${use_gazebo}">
+              <plugin>mock_components/GenericSystem</plugin>
+              </xacro:unless>
+              <xacro:if value="${use_gazebo}">
+                <xacro:if value="${GZ_VERSION == 'classic'}">
+                  <plugin>gazebo_ros2_control/GazeboSystem</plugin>
                 </xacro:if>
-                <xacro:if value="${name== 'GazeboSystem'}">
-                <plugin>gazebo_ros2_control/GazeboSystem</plugin>
+                <xacro:if value="${GZ_VERSION == 'harmonic'}">
+                  <plugin>gz_ros2_control/GazeboSimSystem</plugin>
                 </xacro:if>
+              </xacro:if>
             </hardware>
             <joint name="base_link_to_link1">

File: src/ugv_roarm_moveit/config/roarm_m3/roarm_m3.ros2_control.xacro (robot description, xacro)
@@ -1,14 +1,19 @@
 <?xml version="1.0"?>
 <robot xmlns:xacro="http://www.ros.org/wiki/xacro">
-    <xacro:macro name="roarm_ros2_control" params="name initial_positions_file">
+    <xacro:macro name="roarm_ros2_control" params="use_gazebo GZ_VERSION initial_positions_file">
         <xacro:property name="initial_positions" value="${load_yaml(initial_positions_file)['initial_positions']}"/>
-        <ros2_control name="${name}" type="system">
+        <ros2_control name="RoarmHardware" type="system">
             <hardware>
-                <xacro:if value="${name== 'FakeSystem'}">
-                <plugin>mock_components/GenericSystem</plugin>
+              <xacro:unless value="${use_gazebo}">
+              <plugin>mock_components/GenericSystem</plugin>
+              </xacro:unless>
+              <xacro:if value="${use_gazebo}">
+                <xacro:if value="${GZ_VERSION == 'classic'}">
+                  <plugin>gazebo_ros2_control/GazeboSystem</plugin>
                 </xacro:if>
-                <xacro:if value="${name== 'GazeboSystem'}">
-                <plugin>gazebo_ros2_control/GazeboSystem</plugin>
+                <xacro:if value="${GZ_VERSION == 'harmonic'}">
+                  <plugin>gz_ros2_control/GazeboSimSystem</plugin>
                 </xacro:if>
+              </xacro:if>
             </hardware>
             <joint name="base_link_to_link1">

File: src/ugv_roarm_moveit/config/ugv_roarm.urdf.xacro (robot description, xacro)
@@ -1,9 +1,25 @@
 <?xml version="1.0"?>
 <robot xmlns:xacro="http://www.ros.org/wiki/xacro" name="ugv_roarm">
-<xacro:arg name="ros2_control_plugin" default="FakeSystem"/>
-<xacro:property name="ros2_control_plugin" value="$(arg ros2_control_plugin)"/>
+<xacro:macro name="use_gazebo" params="use_gazebo"></xacro:macro>
+<xacro:arg name="use_gazebo" default="false"/>
+<xacro:property name="use_gazebo" value="$(arg use_gazebo)"/>
+<xacro:macro name="GZ_VERSION" params="GZ_VERSION"></xacro:macro>
+<xacro:arg name="GZ_VERSION" default="classic"/>
+<xacro:property name="GZ_VERSION" value="$(arg GZ_VERSION)"/>
 <xacro:arg name="initial_positions_file" default="$(arg roarm_model)/initial_positions.yaml" />
 <xacro:include filename="$(arg roarm_model)/$(arg roarm_model).ros2_control.xacro" />
-<xacro:roarm_ros2_control name="$(arg ros2_control_plugin)" initial_positions_file="$(arg initial_positions_file)"/>
+<xacro:roarm_ros2_control use_gazebo="$(arg use_gazebo)" GZ_VERSION="$(arg GZ_VERSION)" initial_positions_file="$(arg initial_positions_file)"/>
 <xacro:include filename="$(find ugv_roarm_description)/urdf/ugv_roarm.xacro"/>
+<gazebo>
+    <xacro:if value="${GZ_VERSION == 'classic'}">
+    <plugin filename="libgazebo_ros2_control.so" name="gazebo_ros2_control">
+        <parameters>$(find ugv_roarm_moveit)/config/$(arg roarm_model)/ros2_controllers.yaml</parameters>
+    </plugin>
+    </xacro:if>
+    <xacro:if value="${GZ_VERSION == 'harmonic'}">
+    <plugin name="gz_ros2_control::GazeboSimROS2ControlPlugin" filename="libgz_ros2_control-system.so">
+        <parameters>$(find ugv_roarm_moveit)/config/$(arg roarm_model)/ros2_controllers.yaml</parameters>
+    </plugin>
+    </xacro:if>
+</gazebo>
 </robot>

Commit message: Update the MoveIt plugin.

File: src/ugv_roarm_moveit/config/roarm_m2/roarm_m2.ros2_control.xacro (robot description, xacro)
@@ -38,8 +38,8 @@
                 <state_interface name="velocity"/>
             </joint>
-            <joint name="link3_to_gripper_link">
+            <joint name="gripper_joint">
                 <command_interface name="position"/>
                 <state_interface name="position">
-                  <param name="initial_value">${initial_positions['link3_to_gripper_link']}</param>
+                  <param name="initial_value">${initial_positions['gripper_joint']}</param>
                 </state_interface>
                 <state_interface name="velocity"/>
