Commit message: Roarm M2 adds a gripper.

File: src/ugv_roarm_description/urdf/roarm/bases/roarm_m2.xacro (robot description, xacro)
@@ -7,4 +7,7 @@
 <xacro:arg name="add_camera" default="false"/>
 <xacro:property name="add_camera" value="$(arg add_camera)"/>
+<xacro:macro name="add_depth_camera" params="add_depth_camera"></xacro:macro>
+<xacro:arg name="gripper_type" default="angular_direct"/>
+<xacro:property name="gripper_type" value="$(arg gripper_type)"/>
 <xacro:if value="${add_depth_camera}">
 <xacro:include filename="$(find roarm_description)/urdf/camera/depth_camera.xacro" />
@@ -25,14 +28,18 @@
 <xacro:include filename="$(find roarm_description)/urdf/camera/camera.gazebo.xacro" />
 <xacro:cam use_gazebo="true">
-  <parent link="link3" />
-  <origin xyz="-0.046 -0.183536 0" rpy="1.5708 0 -1.5708" />
-  <!-- <origin xyz="-0.046 -0.172193 0" rpy="1.5708 0 -1.5708" /> -->
-  <!-- usb cam in hand -->
-</xacro:cam>
-<!-- <xacro:cam use_gazebo="true">
-  <parent link="base_link" />
-  <origin xyz="0.06531 0 0.021953" rpy="0 0 0" />
-  usb cam out hand
-</xacro:cam>  -->
+  <xacro:if value="${gripper_type == 'angular_direct'}">
+    <parent link="link3" />
+    <origin xyz="-0.046 -0.183536 0" rpy="1.5708 0 -1.5708" />
+  </xacro:if>
+  <xacro:if value="${gripper_type == 'angular_gear'}">
+    <parent link="link3" />
+    <!-- <origin xyz="-0.046 -0.183536 0" rpy="1.5708 0 -1.5708" /> -->
+    <origin xyz="-0.020898 -0.239246 0" rpy="1.5708 0 -1.5708" />
+    <!-- usb cam in hand -->
+  </xacro:if>
+    <!-- <parent link="base_link" />
+    <origin xyz="0.06531 0 0.021953" rpy="0 0 0" /> -->
+    <!-- usb cam out hand -->
+  </xacro:cam>
 </xacro:if>
 <xacro:include filename="$(find ugv_roarm_description)/urdf/roarm/gazebo/$(arg roarm_model).gazebo"/>
@@ -99,7 +106,7 @@
 <link name="link3">
   <inertial>
-    <origin xyz="0.002 -0.13687 0.0059" rpy="0 0 0" />
-    <mass value="0.0269773" />
-    <inertia ixx="0.000199591" ixy="0" ixz="0" iyy="8.01674E-06" iyz="0" izz="0.000196918" />
+    <origin xyz="-0.0015735 -0.083617 -0.00085" rpy="0 0 0" />
+    <mass value="0.0181535" />
+    <inertia ixx="5.50661E-05" ixy="0" ixz="0" iyy="3.08352E-06" iyz="0" izz="5.43323E-05" />
   </inertial>
   <visual>
@@ -114,24 +121,4 @@
     <geometry>
       <mesh filename="file://$(find roarm_description)/meshes/roarm_m2/link3.stl"  scale="1.0 1.0 1.0"/>
-    </geometry>
-  </collision>
-</link>
-<link name="gripper_link">
-  <inertial>
-    <origin xyz="0.029 0.0027 -0.00078" rpy="0 0 0" />
-    <mass value="0.0028708" />
-    <inertia ixx="5.23216E-07" ixy="0" ixz="0" iyy="1.82071E-06" iyz="0" izz="1.60231E-06" />
-  </inertial>
-  <visual>
-    <origin xyz="0 0 0" rpy="0 0 0" />
-    <geometry>
-      <mesh filename="file://$(find roarm_description)/meshes/roarm_m2/gripper_link.stl"  scale="1.0 1.0 1.0"/>
-    </geometry>
-    <material name="silver"/>
-  </visual>
-  <collision>
-    <origin xyz="0 0 0" rpy="0 0 0" />
-    <geometry>
-      <mesh filename="file://$(find roarm_description)/meshes/roarm_m2/gripper_link.stl"  scale="1.0 1.0 1.0"/>
     </geometry>
   </collision>
@@ -159,16 +146,21 @@
   <limit lower="-1" upper="2.95" effort="0" velocity="0" />
 </joint>
-<joint name="link3_to_gripper_link" type="revolute">
-  <origin xyz="0.002906 -0.21599 -0.00066683" rpy="-1.5708 0 -1.5708" />
-  <parent link="link3" />
-  <child link="gripper_link" />
-  <axis xyz="0 0 1" />
-  <limit lower="0" upper="1.5" effort="0" velocity="0" />
-</joint>
-<joint name="link3_to_hand_tcp" type="fixed">
-  <origin xyz="0.002 -0.2802 0" rpy="1.5708 0 -1.5708" />
-  <parent link="link3" />
-  <child link="hand_tcp" />
-  <axis xyz="0 0 0" />
-</joint>
+<xacro:if value="${gripper_type == 'angular_direct'}">
+  <xacro:include filename="$(find roarm_description)/urdf/gripper/gripper.xacro" />
+  <joint name="link3_to_gripper_base" type="fixed">
+    <origin xyz="0.002906 -0.21599 -0.00066683" rpy="1.5708 0 -1.5708" />
+    <parent link="link3" />
+    <child link="gripper_base" />
+    <axis xyz="0 0 1" />
+  </joint>
+</xacro:if>
+<xacro:if value="${gripper_type == 'angular_gear'}">
+  <xacro:include filename="$(find roarm_description)/urdf/gripper/gripper_a.xacro" />
+  <joint name="link3_to_gripper_base" type="fixed">
+    <origin xyz="-0.002998 -0.186601 -0.000835" rpy="1.5708 0 -1.5708" />
+    <parent link="link3" />
+    <child link="gripper_base" />
+    <axis xyz="0 0 1" />
+  </joint>
+</xacro:if>
 </robot>

Commit message: Precise camera location.

File: src/ugv_roarm_description/urdf/roarm/bases/roarm_m2.xacro (robot description, xacro)
@@ -30,5 +30,5 @@
   <xacro:if value="${gripper_type == 'angular_direct'}">
     <parent link="link3" />
-    <origin xyz="-0.046 -0.183536 0" rpy="1.5708 0 -1.5708" />
+    <origin xyz="-0.062588 -0.181612 0" rpy="1.5708 0 -1.3963" />
   </xacro:if>
   <xacro:if value="${gripper_type == 'angular_gear'}">
