Commit message: Compatible with the new version of Gazebo.

File: src/ugv_roarm_description/urdf/roarm/bases/roarm_m2.xacro (robot description, xacro)
@@ -130,5 +130,5 @@
   <child link="link1" />
   <axis xyz="0 0 1" />
-  <limit lower="-3.1416" upper="3.1416" effort="0" velocity="0" />
+  <limit lower="-3.1416" upper="3.1416" effort="20" velocity="3.14" />
 </joint>
 <joint name="link1_to_link2" type="revolute">
@@ -137,5 +137,5 @@
   <child link="link2" />
   <axis xyz="0 0 1" />
-  <limit lower="-1.5708" upper="1.5708" effort="0" velocity="0" />
+  <limit lower="-1.5708" upper="1.5708" effort="20" velocity="3.14" />
 </joint>
 <joint name="link2_to_link3" type="revolute">
@@ -144,5 +144,5 @@
   <child  link="link3" />
   <axis xyz="0 0 1" />
-  <limit lower="-1" upper="2.95" effort="0" velocity="0" />
+  <limit lower="-1" upper="2.95" effort="20" velocity="3.14" />
 </joint>
 <xacro:if value="${gripper_type == 'angular_direct'}">

File: src/ugv_roarm_description/urdf/roarm/bases/roarm_m3.xacro (robot description, xacro)
@@ -185,6 +185,6 @@
     lower="-3.1416"
     upper="3.1416"
-    effort="0"
-    velocity="0" />
+    effort="20"
+    velocity="3.14" />
 </joint>
 <joint name="link1_to_link2" type="revolute">
@@ -196,6 +196,6 @@
     lower="-1.5708"
     upper="1.5708"
-    effort="0"
-    velocity="0" />
+    effort="20"
+    velocity="3.14" />
 </joint>
 <joint name="link2_to_link3" type="revolute">
@@ -207,6 +207,6 @@
     lower="-1"
     upper="2.95"
-    effort="0"
-    velocity="0" />
+    effort="20"
+    velocity="3.14" />
 </joint>
 <joint name="link3_to_link4" type="revolute">
@@ -218,6 +218,6 @@
     lower="-1.5708"
     upper="1.5708"
-    effort="0"
-    velocity="0" />
+    effort="20"
+    velocity="3.14" />
 </joint>
 <joint name="link4_to_link5" type="revolute">
@@ -229,6 +229,6 @@
     lower="-3.1416"
     upper="3.1416"
-    effort="0"
-    velocity="0" />
+    effort="20"
+    velocity="3.14" />
 </joint>
 <joint name="link5_to_gripper_link" type="revolute">
@@ -240,6 +240,6 @@
     lower="0"
     upper="1.5"
-    effort="0"
-    velocity="0" />
+    effort="20"
+    velocity="3.14" />
 </joint>
 <joint name="link5_to_hand_tcp" type="fixed">

Commit message: Frames (key): Chassis base_link ≠ arm root ugv_roarm_base_link; MTC demos/configs, Cartesian motions, and lift/lower directions use the arm root; Servo planning/command frames set to ugv_roarm_base_link Harmonic hand-eye: Dedicated ugv_roarm_gazebo bridge (chassis cmd_vel/odom/scan + hand cam/image / hand_oak) instead of the chassis-only bridge Launch: MTC demo / Servo forward add_camera; run.launch supports use_sim_time; moveit_gazebo injects robot_description explicitly MoveIt: Hand-eye collision pairs for M2/M3; home pose uses ready (M2 has no observe) Other: navigatetoposecmd uses points_file parameter; ugv_roarm_description declares deps on ugv_description / roarm_description; removed duplicated local UGV base xacros in favor of the overlay Docs: Fixed Frame / arm-root frame notes match the code

File: src/ugv_roarm_description/urdf/roarm/bases/roarm_m2.xacro (robot description, xacro)
@@ -1,27 +1,6 @@
 <?xml version="1.0" ?>
 <robot name="roarm_m2" xmlns:xacro="http://www.ros.org/wiki/xacro">
-<xacro:macro name="add_depth_camera" params="add_depth_camera"></xacro:macro>
-<xacro:arg name="add_depth_camera" default="false"/>
-<xacro:property name="add_depth_camera" value="$(arg add_depth_camera)"/>
-<xacro:macro name="add_camera" params="add_camera"></xacro:macro>
-<xacro:arg name="add_camera" default="false"/>
-<xacro:property name="add_camera" value="$(arg add_camera)"/>
-<xacro:macro name="add_depth_camera" params="add_depth_camera"></xacro:macro>
-<xacro:arg name="gripper_type" default="angular_direct"/>
-<xacro:property name="gripper_type" value="$(arg gripper_type)"/>
-<xacro:if value="${add_depth_camera}">
-<xacro:include filename="$(find roarm_description)/urdf/camera/depth_camera.xacro" />
-<xacro:include filename="$(find roarm_description)/urdf/camera/depth_camera.gazebo.xacro" />
-<!-- <xacro:oak use_gazebo="true">
-  <parent link="link4" />
-  <origin xyz="-0.066257 -0.0523 0" rpy="1.5708 0 -1.5708" />
-  oak cam in hand
-</xacro:oak>   -->
-<xacro:oak use_gazebo="true">
-  <parent link="base_link" />
-  <origin xyz="0.06531 0 0.021953" rpy="0 0 0" />
-  <!-- usb cam out hand -->
-</xacro:oak>
-</xacro:if>
+<!-- add_camera / GZ_VERSION / gripper_type: declared in ugv_roarm.urdf.xacro -->
+<!-- M2 depth-camera mount not designed yet; add_depth_camera is a no-op on M2. -->
 <xacro:if value="${add_camera}">
 <xacro:include filename="$(find roarm_description)/urdf/camera/camera.xacro" />

File: src/ugv_roarm_description/urdf/roarm/bases/roarm_m3.xacro (robot description, xacro)
@@ -1,10 +1,5 @@
 <?xml version="1.0" ?>
 <robot name="roarm_m3" xmlns:xacro="http://www.ros.org/wiki/xacro">
-<xacro:macro name="add_depth_camera" params="add_depth_camera"></xacro:macro>
-<xacro:arg name="add_depth_camera" default="false"/>
-<xacro:property name="add_depth_camera" value="$(arg add_depth_camera)"/>
-<xacro:macro name="add_camera" params="add_camera"></xacro:macro>
-<xacro:arg name="add_camera" default="false"/>
-<xacro:property name="add_camera" value="$(arg add_camera)"/>
+<!-- add_camera / add_depth_camera / GZ_VERSION: declared in ugv_roarm.urdf.xacro -->
 <xacro:if value="${add_depth_camera}">
 <xacro:include filename="$(find roarm_description)/urdf/camera/depth_camera.xacro" />

File: src/ugv_roarm_description/urdf/ugv_roarm.xacro (robot description, xacro)
@@ -3,11 +3,5 @@
 <xacro:arg name="robot_namespace" default="/" />
 <xacro:arg name="urdf_extras" default="empty.urdf" />
-<xacro:arg name="use_gazebo" default="false"/>
-<xacro:arg name="ugv_model" default="ugv_rover"/>
-<xacro:property name="ugv_model" value="$(arg ugv_model)"/>
-<xacro:arg name="roarm_model" default="roarm_m3"/>
-<xacro:property name="roarm_model" value="$(arg roarm_model)"/>
-<xacro:arg name="add_pt" default="false"/>
-<xacro:property name="add_pt" value="$(arg add_pt)"/>
+<!-- Model/feature args are declared once in ugv_roarm.urdf.xacro. -->
 <xacro:include filename="$(find ugv_description)/urdf/bases/$(arg ugv_model).xacro"/>
 <xacro:include filename="$(find ugv_roarm_description)/urdf/roarm/bases/$(arg roarm_model).xacro"/>

File: src/ugv_roarm_moveit/config/roarm_m2/roarm_m2.ros2_control.xacro (robot description, xacro)
@@ -1,5 +1,5 @@
 <?xml version="1.0"?>
 <robot xmlns:xacro="http://www.ros.org/wiki/xacro">
-    <xacro:macro name="roarm_ros2_control" params="use_gazebo GZ_VERSION initial_positions_file">
+    <xacro:macro name="roarm_ros2_control" params="use_gazebo GZ_VERSION gripper_type initial_positions_file">
         <xacro:property name="initial_positions" value="${load_yaml(initial_positions_file)['initial_positions']}"/>
         <ros2_control name="RoarmHardware" type="system">
@@ -45,4 +45,56 @@
                 <state_interface name="velocity"/>
             </joint>
+            <!-- Same as standalone roarm_m2: Harmonic drives finger mimics via gz_ros2_control
+                 (URDF <mimic> alone is not enough for dartsim). -->
+            <xacro:if value="${gripper_type == 'angular_gear'}">
+            <joint name="gripper_left_joint1">
+              <param name="mimic">gripper_joint</param>
+              <param name="multiplier">1</param>
+              <state_interface name="position">
+                <param name="initial_value">${initial_positions['gripper_joint']}</param>
+              </state_interface>
+              <state_interface name="velocity"/>
+            </joint>
+            <joint name="gripper_left_joint2">
+              <param name="mimic">gripper_joint</param>
+              <param name="multiplier">1</param>
+              <state_interface name="position">
+                <param name="initial_value">${initial_positions['gripper_joint']}</param>
+              </state_interface>
+              <state_interface name="velocity"/>
+            </joint>
+            <joint name="gripper_left_joint3">
+              <param name="mimic">gripper_joint</param>
+              <param name="multiplier">-1</param>
+              <state_interface name="position">
+                <param name="initial_value">${initial_positions['gripper_joint']}</param>
+              </state_interface>
+              <state_interface name="velocity"/>
+            </joint>
+            <joint name="gripper_right_joint1">
+              <param name="mimic">gripper_joint</param>
+              <param name="multiplier">1</param>
+              <state_interface name="position">
+                <param name="initial_value">${initial_positions['gripper_joint']}</param>
+              </state_interface>
+              <state_interface name="velocity"/>
+            </joint>
+            <joint name="gripper_right_joint2">
+              <param name="mimic">gripper_joint</param>
+              <param name="multiplier">-1</param>
+              <state_interface name="position">
+                <param name="initial_value">${initial_positions['gripper_joint']}</param>
+              </state_interface>
+              <state_interface name="velocity"/>
+            </joint>
+            <joint name="gripper_right_joint3">
+              <param name="mimic">gripper_joint</param>
+              <param name="multiplier">1</param>
+              <state_interface name="position">
+                <param name="initial_value">${initial_positions['gripper_joint']}</param>
+              </state_interface>
+              <state_interface name="velocity"/>
+            </joint>
+            </xacro:if>
             <joint name="left_down_wheel_link_joint">
                 <state_interface name="position">

File: src/ugv_roarm_moveit/config/ugv_roarm.urdf.xacro (robot description, xacro)
@@ -1,4 +1,5 @@
 <?xml version="1.0"?>
 <robot xmlns:xacro="http://www.ros.org/wiki/xacro" name="ugv_roarm">
+<!-- Single entry-point declarations for the whole ugv_roarm tree. -->
 <xacro:macro name="use_gazebo" params="use_gazebo"></xacro:macro>
 <xacro:arg name="use_gazebo" default="false"/>
@@ -7,7 +8,21 @@
 <xacro:arg name="GZ_VERSION" default="classic"/>
 <xacro:property name="GZ_VERSION" value="$(arg GZ_VERSION)"/>
+<xacro:arg name="ugv_model" default="ugv_rover"/>
+<xacro:property name="ugv_model" value="$(arg ugv_model)"/>
+<xacro:arg name="roarm_model" default="roarm_m2"/>
+<xacro:property name="roarm_model" value="$(arg roarm_model)"/>
+<xacro:arg name="gripper_type" default="angular_direct"/>
+<xacro:property name="gripper_type" value="$(arg gripper_type)"/>
+<xacro:macro name="add_camera" params="add_camera"></xacro:macro>
+<xacro:arg name="add_camera" default="false"/>
+<xacro:property name="add_camera" value="$(arg add_camera)"/>
+<xacro:macro name="add_depth_camera" params="add_depth_camera"></xacro:macro>
+<xacro:arg name="add_depth_camera" default="false"/>
+<xacro:property name="add_depth_camera" value="$(arg add_depth_camera)"/>
+<xacro:arg name="add_pt" default="false"/>
+<xacro:property name="add_pt" value="$(arg add_pt)"/>
 <xacro:arg name="initial_positions_file" default="$(arg roarm_model)/initial_positions.yaml" />
 <xacro:include filename="$(arg roarm_model)/$(arg roarm_model).ros2_control.xacro" />
-<xacro:roarm_ros2_control use_gazebo="$(arg use_gazebo)" GZ_VERSION="$(arg GZ_VERSION)" initial_positions_file="$(arg initial_positions_file)"/>
+<xacro:roarm_ros2_control use_gazebo="$(arg use_gazebo)" GZ_VERSION="$(arg GZ_VERSION)" gripper_type="$(arg gripper_type)" initial_positions_file="$(arg initial_positions_file)"/>
 <xacro:include filename="$(find ugv_roarm_description)/urdf/ugv_roarm.xacro"/>
 <gazebo>
